File: powerboard.sch (EAGLE design)
At the start: 4 parts, among them U1 MCP73831T-2DCI/MC

Commit message: progress
Parts:
- added 3V3OUT, 5V-IN, BAT2+, BAT2-, BAT3+, BAT3-, GND-IN, GNDOUT: (no value), wirepad:2,54/0,9
- added C1, C2: 4.7uF, rcl:C-USC0402
- added C3: 10uF, rcl:C-USC0402
- added C4: 22uF, rcl:C-USC0402
- added IC1: ISL9122AIRNZ-T, ISL9122AIRNZ-T:ISL9122AIRNZ-T
- added JUMPER: 0, rcl:R-US_R0805
- added L1: (no value), rcl:L-USL0201
- added LED1: (no value), led:LEDCHIPLED_0603
- added LEDCURRENT: 0, rcl:R-US_R2512
- added R2: (no value), rcl:R-TRIMMCVR42A
- added RPROG1: 470, rcl:R-US_R0402
- added U$1: CHIPLED, samsung_chipled:CHIPLED
- added U2: MIC826RYMT-TR, mic826rymt-tr:MIC826RYMT-TR
Connections:
- new net 3.3REGULATED: 3V3OUT.P, C4.1, IC1.VOUT, LEDCURRENT.1
- new net 5VIN: 5V-IN.P, C1.1, U1.VDD
- new net BAT_IN: C3.1, IC1.VIN, JUMPER.2, U2.VCC
- new net INDUCTOR1: IC1.LX2, L1.1
- new net INDUCTOR2: IC1.LX1, L1.2
- new net JUMPER: BAT1+.P, BAT2+.P, BAT3+.P, C2.1, JUMPER.1, U1.VBAT
- new net LED+: R2.S, U$1.ANODE
- new net N$10: IC1.EN, U2./RESET
- new net N$2: LEDCURRENT.2, R2.E
- new net N$4: LED1.A, U1.STAT
- new net N$5: LED1.C, RPROG1.2
- net GND: now also BAT2-.P, BAT3-.P, C1.2, C2.2, C3.2, C4.2, GND-IN.P, GNDOUT.P, IC1.EP, IC1.GND, IC1.SCL, IC1.SDA, RPROG1.1, U$1.CATHODE, U1.EXP, U2.GND, U2.GND_2
Other:
- moved on the sheet: BAT1+, BAT1-

Commit message: progress
Parts:
- C1, C2, C3, C4: device rcl:C-USC0402 -> rcl:C-USC0603K
- L1: value (none) -> 1uf; device rcl:L-USL0201 -> vishayinductor:IHHP0806ZHER1R0M01
Connections:
- net INDUCTOR1: now also L1.2; no longer L1.1
- net INDUCTOR2: now also L1.1; no longer L1.2
Changed lines of the file:
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@@
 <part name="GND-IN" library="wirepad" library_urn="urn:adsk.eagle:library:412" deviceset="2,54/0,9" device="" package3d_urn="urn:adsk.eagle:package:30847/1"/>
 <part name="SUPPLY4" library="supply2" library_urn="urn:adsk.eagle:library:372" deviceset="GND" device=""/>
-<part name="C1" library="rcl" library_urn="urn:adsk.eagle:library:334" deviceset="C-US" device="C0402" package3d_urn="urn:adsk.eagle:package:23626/2" value="4.7uF"/>
-<part name="C2" library="rcl" library_urn="urn:adsk.eagle:library:334" deviceset="C-US" device="C0402" package3d_urn="urn:adsk.eagle:package:23626/2" value="4.7uF"/>
+<part name="C1" library="rcl" library_urn="urn:adsk.eagle:library:334" deviceset="C-US" device="C0603K" package3d_urn="urn:adsk.eagle:package:23680/2" value="4.7uF"/>
+<part name="C2" library="rcl" library_urn="urn:adsk.eagle:library:334" deviceset="C-US" device="C0603K" package3d_urn="urn:adsk.eagle:package:23680/2" value="4.7uF"/>
 <part name="SUPPLY5" library="supply2" library_urn="urn:adsk.eagle:library:372" deviceset="GND" device=""/>
 <part name="SUPPLY6" library="supply2" library_urn="urn:adsk.eagle:library:372" deviceset="GND" device=""/>
@@
 <part name="SUPPLY7" library="supply2" library_urn="urn:adsk.eagle:library:372" deviceset="GND" device=""/>
 <part name="IC1" library="ISL9122AIRNZ-T" deviceset="ISL9122AIRNZ-T" device=""/>
-<part name="C3" library="rcl" library_urn="urn:adsk.eagle:library:334" deviceset="C-US" device="C0402" package3d_urn="urn:adsk.eagle:package:23626/2" value="10uF"/>
+<part name="C3" library="rcl" library_urn="urn:adsk.eagle:library:334" deviceset="C-US" device="C0603K" package3d_urn="urn:adsk.eagle:package:23680/2" value="10uF"/>
 <part name="SUPPLY8" library="supply2" library_urn="urn:adsk.eagle:library:372" deviceset="GND" device=""/>
 <part name="SUPPLY9" library="supply2" library_urn="urn:adsk.eagle:library:372" deviceset="GND" device=""/>
-<part name="L1" library="rcl" library_urn="urn:adsk.eagle:library:334" deviceset="L-US" device="L0201" package3d_urn="urn:adsk.eagle:package:23513/2"/>
-<part name="C4" library="rcl" library_urn="urn:adsk.eagle:library:334" deviceset="C-US" device="C0402" package3d_urn="urn:adsk.eagle:package:23626/2" value="22uF"/>
+<part name="C4" library="rcl" library_urn="urn:adsk.eagle:library:334" deviceset="C-US" device="C0603K" package3d_urn="urn:adsk.eagle:package:23680/2" value="22uF"/>
 <part name="SUPPLY10" library="supply2" library_urn="urn:adsk.eagle:library:372" deviceset="GND" device=""/>
 <part name="SUPPLY11" library="supply2" library_urn="urn:adsk.eagle:library:372" deviceset="GND" device=""/>
@@
 <part name="3V3OUT" library="wirepad" library_urn="urn:adsk.eagle:library:412" deviceset="2,54/0,9" device="" package3d_urn="urn:adsk.eagle:package:30847/1"/>
 <part name="GNDOUT" library="wirepad" library_urn="urn:adsk.eagle:library:412" deviceset="2,54/0,9" device="" package3d_urn="urn:adsk.eagle:package:30847/1"/>
+<part name="L1" library="vishayinductor" deviceset="IHHP0806ZHER1R0M01" device="" value="1uf"/>
 </parts>
 <sheets>
@@
 <attribute name="VALUE" x="262.255" y="17.145" size="1.778" layer="96"/>
 </instance>
-<instance part="L1" gate="G$1" x="264.16" y="50.8" smashed="yes" rot="R90">
-<attribute name="NAME" x="269.24" y="49.53" size="1.778" layer="95" rot="R180"/>
-<attribute name="VALUE" x="269.24" y="54.61" size="1.778" layer="96" rot="R180"/>
-</instance>
 <instance part="C4" gate="G$1" x="327.66" y="45.72" smashed="yes">
 <attribute name="NAME" x="328.676" y="46.355" size="1.778" layer="95"/>
@@
 <attribute name="NAME" x="344.043" y="33.7058" size="1.778" layer="95" rot="R180"/>
 <attribute name="VALUE" x="333.883" y="36.322" size="1.778" layer="96" rot="R180"/>
+</instance>
+<instance part="L1" gate="A" x="248.92" y="53.34" smashed="yes">
+<attribute name="VALUE" x="246.9388" y="49.0728" size="3.4798" layer="96" ratio="10" rot="SR0"/>
+<attribute name="NAME" x="248.0056" y="56.6928" size="3.4798" layer="95" ratio="10" rot="SR0"/>
 </instance>
 </instances>
@@
 <segment>
 <pinref part="IC1" gate="G$1" pin="LX1"/>
-<pinref part="L1" gate="G$1" pin="2"/>
-<wire x1="271.78" y1="50.8" x2="274.32" y2="50.8" width="0.1524" layer="91"/>
+<wire x1="264.16" y1="50.8" x2="274.32" y2="50.8" width="0.1524" layer="91"/>
+<pinref part="L1" gate="A" pin="1"/>
+<wire x1="264.16" y1="53.34" x2="264.16" y2="50.8" width="0.1524" layer="91"/>
 </segment>
 </net>
 <net name="INDUCTOR1" class="1">
 <segment>
-<pinref part="L1" gate="G$1" pin="1"/>
-<wire x1="256.54" y1="50.8" x2="251.46" y2="50.8" width="0.1524" layer="91"/>
-<wire x1="251.46" y1="50.8" x2="251.46" y2="45.72" width="0.1524" layer="91"/>
 <pinref part="IC1" gate="G$1" pin="LX2"/>
-<wire x1="251.46" y1="45.72" x2="274.32" y2="45.72" width="0.1524" layer="91"/>
-</segment>
-</net>
+<wire x1="248.92" y1="53.34" x2="248.92" y2="45.72" width="0.1524" layer="91"/>
+<wire x1="248.92" y1="45.72" x2="274.32" y2="45.72" width="0.1524" layer="91"/>
+<pinref part="L1" gate="A" pin="2"/>
+</segment>
+</net>

Commit message: add jlc rules, edit mic826 footprint
Connections:
- net BAT_IN: now also U2./MR
Changed lines of the file:
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@@
 <pinref part="JUMPER" gate="G$1" pin="2"/>
 <wire x1="160.02" y1="58.42" x2="172.72" y2="58.42" width="0.1524" layer="91"/>
+<pinref part="U2" gate="A" pin="/MR"/>
+<wire x1="177.8" y1="38.1" x2="172.72" y2="38.1" width="0.1524" layer="91"/>
+<wire x1="172.72" y1="38.1" x2="172.72" y2="40.64" width="0.1524" layer="91"/>
+<junction x="172.72" y="40.64"/>
 </segment>
 </net>
@@
 </sheet>
 </sheets>
+<errors>
+</errors>
 </schematic>
 </drawing>

Commit message: update powerboard with fixes
Parts:
- removed LEDCURRENT: 0, rcl:R-US_R2512
- R2: device rcl:R-TRIMMCVR42A -> rcl:R-TRIMM3165W
Connections:
- removed net N$2: LEDCURRENT.2, R2.E
- net 3.3REGULATED: now also R2.E; no longer LEDCURRENT.1
Changed lines of the file:
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@@
 <part name="BAT3-" library="wirepad" library_urn="urn:adsk.eagle:library:412" deviceset="2,54/0,9" device="" package3d_urn="urn:adsk.eagle:package:30847/1"/>
 <part name="U$1" library="samsung_chipled" deviceset="CHIPLED" device=""/>
-<part name="R2" library="rcl" library_urn="urn:adsk.eagle:library:334" deviceset="R-TRIMM" device="CVR42A" package3d_urn="urn:adsk.eagle:package:23735/1"/>
-<part name="LEDCURRENT" library="rcl" library_urn="urn:adsk.eagle:library:334" deviceset="R-US_" device="R2512" package3d_urn="urn:adsk.eagle:package:23545/2" value="0"/>
+<part name="R2" library="rcl" library_urn="urn:adsk.eagle:library:334" deviceset="R-TRIMM" device="3165W" package3d_urn="urn:adsk.eagle:package:23723/1"/>
 <part name="JUMPER" library="rcl" library_urn="urn:adsk.eagle:library:334" deviceset="R-US_" device="R0805" package3d_urn="urn:adsk.eagle:package:23553/2" value="0"/>
 <part name="3V3OUT" library="wirepad" library_urn="urn:adsk.eagle:library:412" deviceset="2,54/0,9" device="" package3d_urn="urn:adsk.eagle:package:30847/1"/>
@@
 <attribute name="NAME" x="354.711" y="44.45" size="1.778" layer="95" rot="R90"/>
 <attribute name="VALUE" x="356.87" y="44.45" size="1.778" layer="96" rot="R90"/>
-</instance>
-<instance part="LEDCURRENT" gate="G$1" x="342.9" y="58.42" smashed="yes">
-<attribute name="NAME" x="339.09" y="59.9186" size="1.778" layer="95"/>
-<attribute name="VALUE" x="339.09" y="55.118" size="1.778" layer="96"/>
 </instance>
 <instance part="JUMPER" gate="G$1" x="154.94" y="58.42" smashed="yes">
@@
 <wire x1="327.66" y1="58.42" x2="327.66" y2="50.8" width="0.1524" layer="91"/>
 <junction x="327.66" y="50.8"/>
-<pinref part="LEDCURRENT" gate="G$1" pin="1"/>
-<wire x1="337.82" y1="58.42" x2="327.66" y2="58.42" width="0.1524" layer="91"/>
 <pinref part="3V3OUT" gate="1" pin="P"/>
 <wire x1="330.2" y1="71.12" x2="327.66" y2="71.12" width="0.1524" layer="91"/>
 <wire x1="327.66" y1="71.12" x2="327.66" y2="58.42" width="0.1524" layer="91"/>
 <junction x="327.66" y="58.42"/>
+<pinref part="R2" gate="G$1" pin="E"/>
+<wire x1="360.68" y1="58.42" x2="360.68" y2="53.34" width="0.1524" layer="91"/>
+<wire x1="327.66" y1="58.42" x2="360.68" y2="58.42" width="0.1524" layer="91"/>
 </segment>
 </net>
@@
 </segment>
 </net>
-<net name="N$2" class="1">
-<segment>
-<pinref part="R2" gate="G$1" pin="E"/>
-<pinref part="LEDCURRENT" gate="G$1" pin="2"/>
-<wire x1="347.98" y1="58.42" x2="360.68" y2="58.42" width="0.1524" layer="91"/>
-<wire x1="360.68" y1="58.42" x2="360.68" y2="53.34" width="0.1524" layer="91"/>
-</segment>
-</net>
